Commit message: Fixed URDF nd SRDF

File: interbotix_ros_xscobots/interbotix_xscobot_descriptions/urdf/control.urdf.xacro (robot description, xacro)
@@ -4,5 +4,5 @@
     <hardware>
       <!-- If we are using the actual, physical robot -->
-      <!-- <xacro:if value="${hardware_type == 'actual'}"> -->
+      <xacro:if value="${hardware_type == 'actual'}">
         <plugin>interbotix_xs_ros_control/XSHardwareInterface</plugin>
         <param name="loop_hz">10</param>
@@ -10,9 +10,9 @@
         <param name="gripper_name">gripper</param>
         <param name="joint_states_topic">joint_states</param>
-      <!-- </xacro:if> -->
+      </xacro:if>
       <!-- If doing basic simulation of the robot -->
-      <!-- <xacro:if value="${hardware_type == 'fake'}">
+      <xacro:if value="${hardware_type == 'fake'}">
         <plugin>fake_components/GenericSystem</plugin>
-      </xacro:if> -->
+      </xacro:if>
       <!-- If simulating the robot in Gazebo Classic -->
       <!-- <xacro:if value="${hardware_type == 'gz_classic'}">

File: interbotix_ros_xscobots/interbotix_xscobot_descriptions/urdf/dx400.urdf.xacro (robot description, xacro)
@@ -473,4 +473,31 @@
     </inertial>
   </link>
+  <joint name="ee_gripper" type="fixed">
+    <axis xyz="1 0 0"/>
+    <origin
+      rpy="0 0 0"
+      xyz="0.03 0 0"/>
+    <parent
+      link="$(arg robot_name)/fingers_link"/>
+    <child
+      link="$(arg robot_name)/ee_gripper_link"/>
+  </joint>
+  <link name="$(arg robot_name)/ee_gripper_link">
+    <inertial>
+      <mass value="0.001"/>
+      <inertia
+        ixx="0.001"
+        iyy="0.001"
+        izz="0.001"
+        ixy="0"
+        ixz="0"
+        iyz="0"/>
+    </inertial>
+  </link>
+  <!-- If the AR tag is being used, then add the AR tag mount -->
+  <!-- <xacro:if value="$(arg show_ar_tag)"> -->
+  <!-- <xacro:include filename="$(find interbotix_xscobot_descriptions)/urdf/ar_tag.urdf.xacro"/> -->
+  <!-- </xacro:if> show_ar_tag -->
+  <!-- If the gripper bar is being used, then also add the gripper bar -->
   <joint name="left_finger" type="prismatic">
     <axis xyz="0 0 1"/>

File: interbotix_ros_xscobots/interbotix_xscobot_moveit/config/srdf/dx400.srdf.xacro (robot description, xacro)
@@ -29,11 +29,35 @@
     </group>
     <!--GROUP STATES: Purpose: Define a named state for a particular group, in terms of joint values. This is useful to define states like 'folded arms'-->
+    <group_state name="pose1" group="interbotix_arm">
+        <joint name="j1" value="-0.945"/>
+        <joint name="j2" value="1.663"/>
+        <joint name="j3" value="-2.103"/>
+        <joint name="j4" value="-1.738"/>
+        <joint name="j5" value="0.242"/>
+        <joint name="j6" value="-2.368"/>
+    </group_state>
+    <group_state name="pose2" group="interbotix_arm">
+        <joint name="j1" value="2.839"/>
+        <joint name="j2" value="1.96"/>
+        <joint name="j3" value="-2.29"/>
+        <joint name="j4" value="-1.845"/>
+        <joint name="j5" value="-0.153"/>
+        <joint name="j6" value="1.618"/>
+    </group_state>
+    <group_state name="pose3" group="interbotix_arm">
+        <joint name="j1" value="-1.97"/>
+        <joint name="j2" value="1.668"/>
+        <joint name="j3" value="-2.404"/>
+        <joint name="j4" value="-0.983"/>
+        <joint name="j5" value="-0.228"/>
+        <joint name="j6" value="0.047"/>
+    </group_state>
     <group_state name="sleep" group="interbotix_arm">
-        <joint name="j1" value="0.00"/>
+        <joint name="j1" value="-1.57"/>
         <joint name="j2" value="2.00"/>
         <joint name="j3" value="-2.83"/>
         <joint name="j4" value="-2.46"/>
         <joint name="j5" value="0.0"/>
-        <joint name="j6" value="-1.7"/>
+        <joint name="j6" value="-1.57"/>
     </group_state>
     <group_state name="home" group="interbotix_arm">
